File: ece-196-robot.kicad_pcb (KiCad board)
At the start: 2 copper layers, 64.5 x 35.8 mm, 31 parts, among them J1 Screw_Terminal_01x02, J10 Conn_01x02_Socket, J4 Conn_01x02_Socket, J5 Conn_01x02_Socket, J6 Conn_01x04_Pin, J7 Conn_01x04_Pin, J8 Conn_01x20_Pin, J9 Conn_01x20_Pin, U1 L298N, U2 LM7805_TO220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

Commit message: Update board
Other:
- board text added: "L298N Motor Driver x2"
- board text added: "Motors Pins"
- board text added: "Pins for Devboard"
- board text added: "Power Supply Port"
- board text added: "Ultra Sonic Sensor Pins"
- board text added: "Voltage Regulator"
Changed lines of the file:
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@@
+		)
+	)
+	(gr_text "Power Supply Port"
+		(at 115.12 101.245 90)
+		(layer "Cmts.User")
+		(effects
+			(font
+				(size 1 1)
+				(thickness 0.15)
+			)
+			(justify left bottom)
+		)
+	)
+	(gr_text "Pins for Devboard"
+		(at 127.62 119.495 0)
+		(layer "Cmts.User")
+		(effects
+			(font
+				(size 1 1)
+				(thickness 0.15)
+			)
+			(justify left bottom)
+		)
+	)
+	(gr_text "Motors Pins"
+		(at 181.62 87.245 270)
+		(layer "Cmts.User")
+		(effects
+			(font
+				(size 1 1)
+				(thickness 0.15)
+			)
+			(justify left bottom)
+		)
+	)
+	(gr_text "Pins for Devboard"
+		(at 127.37 81.495 0)
+		(layer "Cmts.User")
+		(effects
+			(font
+				(size 1 1)
+				(thickness 0.15)
+			)
+			(justify left bottom)
+		)
+	)
+	(gr_text "Motors Pins"
+		(at 181.37 98.995 270)
+		(layer "Cmts.User")
+		(effects
+			(font
+				(size 1 1)
+				(thickness 0.15)
+			)
+			(justify left bottom)
+		)
+	)
+	(gr_text "Voltage Regulator"
+		(at 131.87 101.995 90)
+		(layer "Cmts.User")
+		(effects
+			(font
+				(size 1 1)
+				(thickness 0.15)
+			)
+			(justify left bottom)
+		)
+	)
+	(gr_text "L298N Motor Driver x2"
+		(at 137.87 99.995 0)
+		(layer "Cmts.User")
+		(effects
+			(font
+				(size 1 1)
+				(thickness 0.15)
+			)
+			(justify left bottom)
+		)
+	)
+	(gr_text "Ultra Sonic Sensor Pins"
+		(at 111.87 104.495 0)
+		(layer "Cmts.User")
+		(effects
+			(font
+				(size 1 1)
+				(thickness 0.15)
+			)
+			(justify left bottom)
 		)
 	)
